Commit message: add automatically generated frustrum visualization

File: replace_files/robot.urdf.xacro (robot description, xacro)
@@ -3,4 +3,23 @@
   <xacro:arg name="type_name" default="ELISE-UR"/> <!-- ELISE, ELISE-UR, ELISE-CC -->
   <xacro:property name="type" value="$(arg type_name)"/>
+  <!-- ELISE -->
+  <xacro:include filename="$(find elise_description)/urdf/elise.xacro"/>
+  <!-- Sensor Frustum -->
+  <material name="transparent">
+    <color rgba="1.0 1.0 1.0 0.5"/>
+  </material>
+  <link name="sensor_frustum">
+    <visual>
+      <geometry>
+        <mesh filename="package://elise_description/meshes/visual/frustum.STL"/>
+      </geometry>
+      <material name="transparent"/>
+    </visual>
+  </link>
+  <joint name="sensor_frustum_joint" type="fixed">
+    <origin xyz="0 0 0" rpy="0 0 0" />
+    <parent link="end_effector"/>
+    <child link="sensor_frustum" />
+  </joint>
   <!-- Add base link if only the ELISE is used -->
   <xacro:if value="${type == 'ELISE'}">
@@ -12,9 +31,10 @@
     </joint>
   </xacro:if>
-  <xacro:include filename="$(find elise_description)/urdf/elise.xacro"/>
   <xacro:if value="${type == 'ELISE-UR'}">
+    <!-- UR-10 -->
     <xacro:include filename="$(find elise_description)/urdf/elise_ur10.xacro"/>
   </xacro:if>
   <xacro:if value="${type == 'ELISE-CC'}">
+    <!-- Cartesian Container System -->
     <xacro:include filename="$(find elise_description)/urdf/elise_cc.xacro"/>
   </xacro:if>

Commit message: use argpars to provide arguments

File: replace_files/robot.urdf.xacro (robot description, xacro)
@@ -37,5 +37,10 @@
   <xacro:if value="${type == 'ELISE-CC'}">
     <!-- Cartesian Container System -->
-    <xacro:include filename="$(find elise_description)/urdf/elise_cc.xacro"/>
+    <xacro:include filename="$(find container_description)/urdf/container.xacro"/>
+    <joint name="tool_joint" type="fixed">
+      <origin xyz="0 0 0" rpy="0 0 0" />
+      <parent link="tool0"/>
+      <child link="endo_box" />
+    </joint>
   </xacro:if>
 </robot>

Commit message: add parameters for link lengths

File: replace_files/robot.urdf.xacro (robot description, xacro)
@@ -3,6 +3,4 @@
   <xacro:arg name="type_name" default="ELISE-UR"/> <!-- ELISE, ELISE-UR, ELISE-CC -->
   <xacro:property name="type" value="$(arg type_name)"/>
-  <!-- ELISE -->
-  <xacro:include filename="$(find elise_description)/urdf/elise.xacro"/>
   <!-- Sensor Frustum -->
   <material name="transparent">
@@ -24,4 +22,7 @@
   <!-- Add base link if only the ELISE is used -->
   <xacro:if value="${type == 'ELISE'}">
+    <xacro:property name="L1" value="0.4"/>
+    <xacro:property name="L2" value="0.1"/>
+    <xacro:property name="L3" value="0.05"/>
     <link name="base_link"/>
     <joint name="base_joint" type="fixed">
@@ -33,8 +34,14 @@
   <xacro:if value="${type == 'ELISE-UR'}">
     <!-- UR-10 -->
+    <xacro:property name="L1" value="0.4"/>
+    <xacro:property name="L2" value="0.1"/>
+    <xacro:property name="L3" value="0.05"/>
     <xacro:include filename="$(find elise_description)/urdf/elise_ur10.xacro"/>
   </xacro:if>
   <xacro:if value="${type == 'ELISE-CC'}">
     <!-- Cartesian Container System -->
+    <xacro:property name="L1" value="1.6"/>
+    <xacro:property name="L2" value="0.1"/>
+    <xacro:property name="L3" value="0.05"/>
     <xacro:include filename="$(find container_description)/urdf/container.xacro"/>
     <joint name="tool_joint" type="fixed">
@@ -44,3 +51,5 @@
     </joint>
   </xacro:if>
+    <!-- ELISE -->
+  <xacro:include filename="$(find elise_description)/urdf/elise.xacro"/>
 </robot>
